File: dual-mcp3201-pmod.kicad_pcb (KiCad board)
At the start: 2 copper layers, 50 x 20 mm, 34 parts, among them X1 AUB-13, X2 PMOD_PERIPH, X3 RIGHT, X4 LEFT

Commit message: Connect flying via to ground
Routing:
- net GND: vias 17 -> 18
- net (no net): vias 1 -> 0
