File: dual-mcp3201-pmod.sch (KiCad schematic (older format))
At the start: 33 parts, among them X1 AUB-13, X2 PMOD_PERIPH, X3 RIGHT, X4 LEFT

Commit message: Change filter cut-off frequency to 10kHz
Parts:
- C1, C8: value 68p -> 680p
- C10, C3: value 220p -> 2200p
Changed lines of the file:
@@
 P 5200 2850
 F 0 "C1" V 5253 2742 60  0000 R CNN
-F 1 "68p" V 5147 2742 60  0000 R CNN
+F 1 "680p" V 5147 2742 60  0000 R CNN
 F 2 "Capacitor_SMD:C_0603_1608Metric_Pad1.05x0.95mm_HandSolder" H 5200 2850 60  0001 C CNN
 F 3 "" H 5100 2925 60  0000 C CNN
@@
 P 4600 3800
 F 0 "C3" V 4653 3692 60  0000 R CNN
-F 1 "220p" V 4547 3692 60  0000 R CNN
+F 1 "2200p" V 4547 3692 60  0000 R CNN
 F 2 "Capacitor_SMD:C_0603_1608Metric_Pad1.05x0.95mm_HandSolder" H 4600 3800 60  0001 C CNN
 F 3 "" H 4500 3875 60  0000 C CNN
@@
 P 5200 5450
 F 0 "C8" V 5253 5342 60  0000 R CNN
-F 1 "68p" V 5147 5342 60  0000 R CNN
+F 1 "680p" V 5147 5342 60  0000 R CNN
 F 2 "Capacitor_SMD:C_0603_1608Metric_Pad1.05x0.95mm_HandSolder" H 5200 5450 60  0001 C CNN
 F 3 "" H 5100 5525 60  0000 C CNN
@@
 P 4600 6400
 F 0 "C10" V 4653 6292 60  0000 R CNN
-F 1 "220p" V 4547 6292 60  0000 R CNN
+F 1 "2200p" V 4547 6292 60  0000 R CNN
 F 2 "Capacitor_SMD:C_0603_1608Metric_Pad1.05x0.95mm_HandSolder" H 4600 6400 60  0001 C CNN
 F 3 "" H 4500 6475 60  0000 C CNN
